File: Hardware/OpenBook.sch (EAGLE design)
At the start: 103 parts, among them IC1 BD5229G-TR, IC4 XC6220A331MR-G, J1 FH34SRJ-24S-0.5SH_99_, J2 SAMACSYS_PARTS_USB4110-GF-A, J3 QWIIC_RIGHT_ANGLE, J4 112A-TAAR-R03_ATTEND, Q1 20V/4.2A/52mΩ/1.4W, Q2 20V/4.2A/52mΩ/1.4W, Q3 SI1308EDL-T1-GE3, U1 W25Q512JVEIQ, U2 ESP32-C6-WROOM-1-N8, U3 DS3231SN#, U4 MAX17048G+T10

Commit message: Added the project.
Signed-off-by: Cristian-Stefan Lazar <cristian.lazar1512@gmail.com>
Parts:
- removed C10: 100nF, DeskAssistant v19 v1:ESP32_WROVER_EAGLE-LTSPICE_CC0402
- removed C1_BAT2, C5_USB: 4.7uF, DeskAssistant v19 v1:ESP32_WROVER_EAGLE-LTSPICE_CC0402
- removed EPD_C11, EPD_C12: 1uF/50V, DeskAssistant v19 v1:ESP32_WROVER_EAGLE-LTSPICE_CC0402
- removed R1_PINH: 10K, DeskAssistant v19 v1:ESP32_WROVER_EAGLE-LTSPICE_RR0402
- removed R2-USB: 5k1, DeskAssistant v19 v1:ESP32_WROVER_EAGLE-LTSPICE_RR0402
- added C1_BAT: 4.7uF, DeskAssistant v19 v1:ESP32_WROVER_EAGLE-LTSPICE_C0402
- added C3_USB: 100nF, DeskAssistant v19 v1:ESP32_WROVER_EAGLE-LTSPICE_C0402
- added C_TANT: 100uF, DeskAssistant v19 v1:RCL_CPOL-EUCT3528
- added EPD_C3: 0.1uF/50V, DeskAssistant v19 v1:ESP32_WROVER_EAGLE-LTSPICE_C0402
- added EPD_C4: 1uF/50V, DeskAssistant v19 v1:ESP32_WROVER_EAGLE-LTSPICE_C0402
- added R1_PINH2: 10K, DeskAssistant v19 v1:ESP32_WROVER_EAGLE-LTSPICE_RR0402
- added R1_USB: 5k1, DeskAssistant v19 v1:ESP32_WROVER_EAGLE-LTSPICE_RR0402
- C1, C1_BAT1, C2, C2_BAT, C2_BAT1, C8, C9, C_DELAY, EPD_C1, EPD_C10, EPD_C2, EPD_C6, EPD_C7, EPD_C8, EPD_C9: device DeskAssistant v19 v1:ESP32_WROVER_EAGLE-LTSPICE_CC0402 -> DeskAssistant v19 v1:ESP32_WROVER_EAGLE-LTSPICE_C0402
- C3: value 100uF -> 4.7uF/25V; device DeskAssistant v19 v1:RCL_CPOL-EUCT3528 -> DeskAssistant v19 v1:ESP32_WROVER_EAGLE-LTSPICE_C0402
- C4: value 4.7uF/25V -> 1uF; device DeskAssistant v19 v1:ESP32_WROVER_EAGLE-LTSPICE_CC0402 -> DeskAssistant v19 v1:ESP32_WROVER_EAGLE-LTSPICE_C0402
- C4_USB: value 100nF -> 4.7uF; device DeskAssistant v19 v1:ESP32_WROVER_EAGLE-LTSPICE_CC0402 -> DeskAssistant v19 v1:ESP32_WROVER_EAGLE-LTSPICE_C0402
- C5: value 1uF -> 100nF; device DeskAssistant v19 v1:ESP32_WROVER_EAGLE-LTSPICE_CC0402 -> DeskAssistant v19 v1:ESP32_WROVER_EAGLE-LTSPICE_C0402
- C6: value 100nF -> 10uF; device DeskAssistant v19 v1:ESP32_WROVER_EAGLE-LTSPICE_CC0402 -> DeskAssistant v19 v1:ESP32_WROVER_EAGLE-LTSPICE_C0402
- C7: value 10uF -> 100nF; device DeskAssistant v19 v1:ESP32_WROVER_EAGLE-LTSPICE_CC0402 -> DeskAssistant v19 v1:ESP32_WROVER_EAGLE-LTSPICE_C0402
- D1: FF (none) -> FF
- EPD_C5: value 0.1uF/50V -> 1uF/50V; device DeskAssistant v19 v1:ESP32_WROVER_EAGLE-LTSPICE_CC0402 -> DeskAssistant v19 v1:ESP32_WROVER_EAGLE-LTSPICE_C0402
- Q1, Q2: PROD_ID (none) -> DMG2305UX-7
- TP1: TP_SIGNAL_NAME (none) -> TX
- TP10: TP_SIGNAL_NAME (none) -> EPD_CS
- TP11: TP_SIGNAL_NAME (none) -> EPD_DC
- TP12: TP_SIGNAL_NAME (none) -> EPD_RST
- TP13: TP_SIGNAL_NAME (none) -> EPD_3V3_c
- TP14: TP_SIGNAL_NAME (none) -> VBUS
- TP15: TP_SIGNAL_NAME (none) -> INT_RTC
- TP16: TP_SIGNAL_NAME (none) -> 3V3
- TP17: TP_SIGNAL_NAME (none) -> EPD_3V3
- TP2: TP_SIGNAL_NAME (none) -> RX
- TP3: TP_SIGNAL_NAME (none) -> VBAT
- TP4, TP5: TP_SIGNAL_NAME (none) -> GND
- TP6: TP_SIGNAL_NAME (none) -> MISO
- TP7: TP_SIGNAL_NAME (none) -> MOSI
- TP8: TP_SIGNAL_NAME (none) -> SCK
- TP9: TP_SIGNAL_NAME (none) -> EPD_BUSY
- U1: value W25Q512JVEIQ -> ESP32-C6-WROOM-1-N8; device DeskAssistant v19 v1:W25Q512JVEIQ -> DeskAssistant v19 v1:ESP32-C6-WROOM-1-N8
- U2: value ESP32-C6-WROOM-1-N8 -> MAX17048G+T10; device DeskAssistant v19 v1:ESP32-C6-WROOM-1-N8 -> DeskAssistant v19 v1:MAX17048G+T10
- U4: value MAX17048G+T10 -> W25Q512JVEIQ; device DeskAssistant v19 v1:MAX17048G+T10 -> DeskAssistant v19 v1:W25Q512JVEIQ
- U7: value ESP32_WROVER_SPARKFUN-IC-POWER_MCP73831 -> MCP73831
- renumbered C10_SUPERCAP to C_SUPERCAP, IC1 to U6, IC4 to U5, MCP73831 to U7, R1_PWRUSB to R_PWRUSB, R2-PINH to R2-PINH1, R2-USB1 to R2_USB, R2_PINH1 to R2_PINH2, SENSOR2 to U8
Connections:
- removed net GRD: Q3.G, R4.2
- removed net N$12: D10.2, D11.2, D12.2, D6.2, D8.2, D9.2, R10.1, R5.1, R6.1, R7.1, R8.1, R9.1
- new net N$13: R2_BAT.2, U7.PROG
- net 32KHZ: now also U1.IO1; no longer U2.IO1
- net 3V3: now also C2_BAT1.1, C8.1, C_TANT.+, R1_PINH2.2, U1.3V3, U4.!HOLD!/!RESET!(IO3), U4.!WP!(IO2), U4.VCC; no longer C1_BAT2.1, C3.+, C9.1, R1_PINH1.2, U1.!HOLD!/!RESET!(IO3), U1.!WP!(IO2), U1.VCC, U2.3V3
- net EPD_3V3: now also C6.1, EPD_C3.2; no longer C7.1, EPD_C5.2
- net EPD_3V3_C: now also U1.IO20; no longer U2.IO20
- net EPD_BUSY: now also U1.IO3; no longer U2.IO3
- net EPD_CS: now also D6.2, R9.1, U1.IO10; no longer U2.IO10
- net EPD_DC: now also U1.IO5; no longer U2.IO5
- net EPD_RST: now also U1.IO23; no longer U2.IO23
- net FLASH_CS: now also D9.2, R5.1, U1.IO11, U4.!CS; no longer U1.!CS, U2.IO11
- net GDR: now also Q3.G, R4.2
- net GND: now also C1_BAT.2, C3_USB.2, C4.2, C_TANT.-, EPD_C3.1, EPD_C4.1, R1_USB.2, U2.CTG, U2.EP, U2.QSTRT, U4.EXP; no longer C10.2, C1_BAT2.2, C3.-, C5_USB.2, EPD_C11.1, EPD_C12.1, R2-USB.2, U1.EXP, U4.CTG, U4.EP, U4.QSTRT
- net GPIO8: now also U1.IO8; no longer U2.IO8
- net I2C_PW: now also R1_PINH1.2, U1.IO19; no longer R1_PINH.2, U2.IO19
- net INT_RTC: now also R1_PINH2.1, U1.IO0; no longer R1_PINH1.1, U2.IO0
- net IO/BOOT: now also C5.1, U1.IO9; no longer C6.1, U2.IO9
- net IO/CHANGE: now also C9.1, U1.IO15; no longer C10.1, U2.IO15
- net MISO: now also D12.2, R8.1, U1.IO2, U4.DO(IO1); no longer U1.DO(IO1), U2.IO2
- net MOSI: now also D11.2, R7.1, U1.IO7, U4.DI(IO0); no longer U1.DI(IO0), U2.IO7
- net N$10: now also EPD_C6.2; no longer EPD_C8.2
- net N$11: now also EPD_C4.2; no longer EPD_C6.2
- net N$14: now also EPD_C5.2; no longer EPD_C7.2
- net N$15: now also EPD_C10.2; no longer EPD_C12.2
- net N$3: now also C3.1; no longer C4.1
- net N$7: now also R1_USB.1; no longer R2-USB.1
- net N$9: now also EPD_C8.2; no longer EPD_C10.2
- net PREVGH: now also EPD_C7.2; no longer EPD_C9.2
- net PREVGL: now also EPD_C9.2; no longer EPD_C11.2
- net RESET: now also C4.1, U1.EN; no longer C5.1, U2.EN
- net RTC_RST: now also U1.IO18; no longer U2.IO18
- net RX: now also U1.RXD0/GPIO17; no longer TP1.TP, U2.RXD0/GPIO17
- net SCK: now also D10.2, R6.1, U1.IO6, U4.CLK; no longer U1.CLK, U2.IO6
- net SCL: now also U1.IO22, U2.SCL; no longer U2.IO22, U4.SCL
- net SDA: now also R1_PINH1.1, U1.IO21, U2.SDA; no longer R1_PINH.1, U2.IO21, U4.SDA
- net SRC: now also C3.2; no longer C4.2
- net SS_SD: now also D8.2, R10.1, U1.IO4; no longer U2.IO4
- net TX: now also TP1.TP, U1.TXD0/GPIO16; no longer U2.TXD0/GPIO16
- net USB_D+: now also U1.IO13; no longer U2.IO13
- net USB_D-: now also U1.IO12; no longer U2.IO12
- net VBAT: now also U2.CELL, U2.VDD; no longer R2_BAT.2, U4.CELL, U4.VDD, U7.PROG
- net VBUS: now also C1_BAT.1, C3_USB.1; no longer C2_BAT1.1, C5_USB.1, J2.A4, PFMF.050.1.1
- net VRTC: now also C7.1; no longer C8.1
- net VUSB: now also J2.A4, PFMF.050.1.1
Other:
- moved on the sheet: C2_BAT1, C4, C4_USB, C5, C6, C7, C8, C9, D3, D4, EPD_C10, EPD_C5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

Commit message: Fixes #2, fixes #3; Adds the frame and module names in the schematic
Signed-off-by: Cristian-Stefan Lazar <cristian.lazar1512@gmail.com>
Other:
- note added: "Battery Charge Level"
- note added: "Display Type Selector"
- note added: "E-Paper Display Header"
- note added: "E-Paper Drive Circuit"
- note added: "EPD Power"
- note added: "ESP32 C6"
- note added: "Environmental Sensor BME688"
- note added: "External NOR Flash 64MB"
- note added: "LDO Voltage Regulator"
- note added: "Li-Po Battery Charging Controller"
- note added: "Qwiic / Stemma QT"
- note added: "RTC Module DS3231SN"
- note added: "SD Card"
- note added: "SPI ESD Protection Lines"
- note added: "Test Pads"
- note added: "USB C Connector & ESD Protection"
- note added: "Voltage Supervisor + Reset & Boot / IO Button"
- moved on the sheet: BOOT_BUTTON, C1, C1_BAT, C1_BAT1, C2, C2_BAT, C2_BAT1, C3, C3_USB, C4, C4_USB, C5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
